File: hardware/txe8116-module/kicad/txe8116-module.kicad_pcb (KiCad board)
At the start: 4 copper layers, 15.2 x 30.5 mm, 28 parts, among them J1 Conn_01x12, J2 Conn_01x12, U1 TXE8116

Commit message: fix(hardware): add 10k pull-up resistors on RESET and INT per datasheet
Parts:
- added R1: 10k, Resistor_SMD:R_0603_1608Metric, F.Cu at (151.1, 71.3)
- added R2: 10k, Resistor_SMD:R_0603_1608Metric, F.Cu at (149.5, 71.3)
Routing:
- net VCC: track 17.7 -> 21.9 mm, vias 2 -> 3
- net /~{RESET}: track 14.9 -> 16.6 mm
- net /~{INT}: track 10.8 -> 12.0 mm
- net GND: vias 45 -> 47
